Commit message: Fix for HoloOcean offset bug

File: coug_ws/src/coug_description/urdf/bluerov2_holoocean/bluerov2_holoocean.urdf.xacro (robot description, xacro)
@@ -62,5 +62,5 @@
   </joint>
   <link name="sonar_link"/>
-  <!-- Fix for matching CougUV URDF -->
+  <!-- Fixes for matching CougUV URDF -->
   <joint name="modem_joint" type="fixed">
     <parent link="com_link"/>
@@ -69,3 +69,9 @@
   </joint>
   <link name="modem_link"/>
+  <joint name="truth_joint" type="fixed">
+    <parent link="base_link"/>
+    <child link="truth_link"/>
+    <origin xyz="0 0 0" rpy="0 0 0"/>
+  </joint>
+  <link name="truth_link"/>
 </robot>

File: coug_ws/src/coug_description/urdf/couguv_holoocean.urdf.xacro (robot description, xacro)
@@ -127,5 +127,5 @@
     <parent link="base_link"/>
     <child link="com_link"/>
-    <origin xyz="0.0 0 0.0" rpy="0 0 0"/>
+    <origin xyz="0 0 0" rpy="0 0 0"/>
   </joint>
   <link name="com_link"/>
@@ -158,3 +158,10 @@
   </joint>
   <link name="dvl_link"/>
+  <!-- TODO: Fix this in HoloOcean -->
+  <joint name="truth_joint" type="fixed">
+    <parent link="base_link"/>
+    <child link="truth_link"/>
+    <origin xyz="-0.1 0 -0.1" rpy="0 0 0"/>
+  </joint>
+  <link name="truth_link"/>
 </robot>
