Commit message: Added BlueROV2 GPS lever arm

File: coug_ws/src/coug_description/urdf/bluerov2_heavy/bluerov2_heavy.urdf.xacro (robot description, xacro)
@@ -25,4 +25,11 @@
     <origin xyz="0 0 0" rpy="0 0 0"/>
   </joint>
+  <!-- GPS Link -->
+  <link name="gps_link"/>
+  <joint name="gps_joint" type="fixed">
+    <parent link="base_link"/>
+    <child link="gps_link"/>
+    <origin xyz="-0.11770 -0.20723 0.40019" rpy="0 0 0"/>
+  </joint>
   <!-- DVL Link -->
   <link name="dvl_link"/>

Commit message: Cleaner bag launch setup

File: coug_ws/src/coug_description/urdf/bluerov2_heavy/bluerov2_heavy.urdf.xacro (robot description, xacro)
@@ -25,4 +25,11 @@
     <origin xyz="0 0 0" rpy="0 0 0"/>
   </joint>
+  <!-- Depth Link -->
+  <link name="depth_link"/>
+  <joint name="depth_joint" type="fixed">
+    <parent link="base_link"/>
+    <child link="depth_link"/>
+    <origin xyz="0 0 0" rpy="0 0 0"/>
+  </joint>
   <!-- GPS Link -->
   <link name="gps_link"/>
