Commit message: Naming update

File: packages/coug_description/urdf/bluerov2/bluerov2.urdf.xacro (robot description, xacro)
@@ -2,6 +2,6 @@
 <robot xmlns:xacro="http://www.ros.org/wiki/xacro" name="bluerov2">
   <!--
-  @file bluerov2_heavy.urdf.xacro
-  @brief URDF description for the BlueROV2 Heavy configuration.
+  @file bluerov2.urdf.xacro
+  @brief URDF description for the BlueROV2.
   @author Nelson Durrant
   @date Jan 2026
@@ -14,5 +14,5 @@
     <visual>
       <geometry>
-        <mesh filename="package://coug_description/urdf/bluerov2_heavy/meshes/bluerov2_heavy.dae" scale="0.025 0.025 0.025"/>
+        <mesh filename="package://coug_description/urdf/bluerov2/meshes/bluerov2.dae" scale="0.025 0.025 0.025"/>
       </geometry>
     </visual>
